File: Hardware/Baseboard/FPGA4RISCV_BB.kicad_pcb (KiCad board)
At the start: 2 copper layers, 42 parts, among them J1 1473005-4, J2 Conn_02x06_Odd_Even, J3 USB_C_Receptacle_USB2.0_16P, J4 21992304, U2 FT2232HL, Y1 12MHz

Commit message: BB: PCIe update
Parts:
- added C18: 100nF, Capacitor_SMD:C_0402_1005Metric, F.Cu at (127.7, 97.2)
- added C19: 10uF, Capacitor_SMD:C_0402_1005Metric, F.Cu at (127.7, 99.2)
- added C20: 100nF, Capacitor_SMD:C_0402_1005Metric, F.Cu at (127.7, 101.2)
- added C21: 100nF, Capacitor_SMD:C_0402_1005Metric, F.Cu at (127.7, 103.1)
- added C22: 100nF, Capacitor_SMD:C_0402_1005Metric, F.Cu at (127.7, 105.1)
- added C23: 10uF, Capacitor_SMD:C_0402_1005Metric, F.Cu at (127.7, 107.1)
- added C24: 100nF, Capacitor_SMD:C_0402_1005Metric, F.Cu at (130.6, 97.2)
- added C25: 10uF, Capacitor_SMD:C_0402_1005Metric, F.Cu at (130.6, 99.2)
- added C26: 100nF, Capacitor_SMD:C_0402_1005Metric, F.Cu at (130.6, 101.2)
- added C27: 100nF, Capacitor_SMD:C_0402_1005Metric, F.Cu at (130.6, 103.1)
- added C28: 100nF, Capacitor_SMD:C_0402_1005Metric, F.Cu at (130.6, 105.1)
- J4: value 21992304 -> MDT275M02001; footprint FPGA4RISCV:TE_21992304 -> FPGA4RISCV:MDT275M02001
- moved J2 13.9 mm to (155.7, 86.1)
- moved J4 12.6 mm to (138.8, 90.2)
- moved C2 12.4 mm to (111.9, 100.7)
- moved J1 12.4 mm to (133.1, 67.2)
- moved C1 12.4 mm to (111.9, 98.7)
- moved C3 12.4 mm to (111.9, 102.7)
- moved C4 12.4 mm to (111.9, 104.6)
- moved C5 12.4 mm to (111.9, 106.6)
- moved C6 12.4 mm to (111.9, 108.6)
- moved C14 12.4 mm to (117.6, 100.7)
- moved C8 12.4 mm to (114.7, 100.7)
- moved R1 12.4 mm to (111.9, 84.8)
- moved R15 12.4 mm to (117.7, 84.8)
- moved R8 12.4 mm to (114.8, 84.8)
- moved C10 12.4 mm to (114.7, 104.6)
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Connections:
- J4 pad 1: unconnected-(J4-Pad1) -> GND
- J4 pad 11: unconnected-(J4-Pad11) -> PCIe_TX3_N
- J4 pad 12: unconnected-(J4-Pad12) -> +3.3V_PCIe
- J4 pad 13: unconnected-(J4-Pad13) -> PCIe_TX3_P
- J4 pad 14: unconnected-(J4-Pad14) -> +3.3V_PCIe
- J4 pad 15: unconnected-(J4-Pad15) -> GND
- J4 pad 16: unconnected-(J4-Pad16) -> +3.3V_PCIe
- J4 pad 17: unconnected-(J4-Pad17) -> PCIe_RX2_N
- J4 pad 18: unconnected-(J4-Pad18) -> +3.3V_PCIe
- J4 pad 19: unconnected-(J4-Pad19) -> PCIe_RX2_P
- J4 pad 2: unconnected-(J4-Pad2) -> +3.3V_PCIe
- J4 pad 21: unconnected-(J4-Pad21) -> GND
- J4 pad 23: unconnected-(J4-Pad23) -> PCIe_TX2_N
- J4 pad 3: unconnected-(J4-Pad3) -> GND
- J4 pad 33: unconnected-(J4-Pad33) -> GND
- J4 pad 35: unconnected-(J4-Pad35) -> PCIe_TX1_N
- J4 pad 37: unconnected-(J4-Pad37) -> PCIe_TX1_P
- J4 pad 39: unconnected-(J4-Pad39) -> GND
- J4 pad 4: unconnected-(J4-Pad4) -> +3.3V_PCIe
- J4 pad 41: unconnected-(J4-Pad41) -> PCIe_RX0_N
- J4 pad 43: unconnected-(J4-Pad43) -> PCIe_RX0_P
- J4 pad 45: unconnected-(J4-Pad45) -> GND
- J4 pad 47: unconnected-(J4-Pad47) -> PCIe_TX0_N
- J4 pad 49: unconnected-(J4-Pad49) -> PCIe_TX0_P
- J4 pad 5: unconnected-(J4-Pad5) -> PCIe_RX3_N
- J4 pad 50: unconnected-(J4-Pad50) -> PERST#
- J4 pad 51: unconnected-(J4-Pad51) -> GND
- J4 pad 52: unconnected-(J4-Pad52) -> CLKREQ#
- J4 pad 53: unconnected-(J4-Pad53) -> PCIe_CLK_N
- J4 pad 55: unconnected-(J4-Pad55) -> PCIe_CLK_P
- J4 pad 57: unconnected-(J4-Pad57) -> GND
- J4 pad 7: unconnected-(J4-Pad7) -> PCIe_RX3_P
- J4 pad 70: unconnected-(J4-Pad70) -> +3.3V_PCIe
- J4 pad 71: unconnected-(J4-Pad71) -> GND
- J4 pad 72: unconnected-(J4-Pad72) -> +3.3V_PCIe
- J4 pad 73: unconnected-(J4-Pad73) -> GND
- J4 pad 74: unconnected-(J4-Pad74) -> +3.3V_PCIe
- J4 pad 75: unconnected-(J4-Pad75) -> GND
- J4 pad 9: unconnected-(J4-Pad9) -> GND
