File: Hardware/Baseboard/ps.kicad_sch (KiCad schematic)
At the start: 1 part, among them U1 LFE5UM5G-85F-8BG381x

Commit message: SOM board outline
Parts:
- removed U1: LFE5UM5G-85F-8BG381x, Package_BGA:Lattice_caBGA-381_17.0x17.0mm_Layout20x20_P0.8mm_Ball0.4mm_Pad0.4mm_NSMD, symbol FPGA_Lattice:LFE5UM5G-85F-8BG381x

Commit message: BB schematics: PS
Parts:
- added C2, C45: 100nF, Capacitor_SMD:C_0402_1005Metric, symbol RA8M1:885012205092
- added C37, C38, C39, C40: 47uF, Capacitor_SMD:C_2220_5750Metric_Pad1.97x5.40mm_HandSolder, symbol RA8M1:885012205092
- added C41: 22nF, Capacitor_SMD:C_2220_5750Metric_Pad1.97x5.40mm_HandSolder, symbol RA8M1:885012205092
- added C42: 10uF, Capacitor_SMD:C_1210_3225Metric, symbol RA8M1:885012205092
- added C43, C44: 2.2uF, Diode_SMD:D_1206_3216Metric, symbol RA8M1:885012205092
- added D2: PMEG45A10, Package_TO_SOT_SMD:Nexperia_CFP15_SOT-1289, symbol Diode:PMEG45A10EPD
- added J6: Barrel_Jack_Switch, symbol Connector:Barrel_Jack_Switch
- added JP1: PS_DIS, symbol Jumper:SolderJumper_2_Open
- added L4: 8.2uH, symbol Device:L
- added R28: 86.6k, Resistor_SMD:R_0402_1005Metric, symbol Device:R
- added R29: FBT-56k, Resistor_SMD:R_0402_1005Metric, symbol Device:R
- added R30: FBB-10k, Resistor_SMD:R_0402_1005Metric, symbol Device:R
- added U3: LV14540DDAR, SOIC127P600X170-9N, symbol FPGA4RISCV:LV14540DDAR
Connections:
- new net: C42.2, C43.2, C44.2, C45.2, J6.1, U3.2 (VIN)
- new net: R29.2, R30.1, U3.5 (FB)
- new net: C2.1, U3.1 (BOOT)
- new net: JP1.2 (B), U3.3 (EN)
- new net: R28.1, U3.4 (RT/SYNC)
- new net: C41.2, U3.6 (SS)
- new net: C2.2, D2.3 (K), L4.1, U3.8 (SW)
- new net +5V_PS: C37.2, C38.2, C39.2, C40.2, L4.2, R29.1
- new net GND: C37.1, C38.1, C39.1, C40.1, C41.1, C42.1, C43.1, C44.1, C45.1, D2.1 (A), D2.2 (A), J6.2, JP1.1 (A), R28.2, R30.2, U3.7 (GND), U3.9 (EP)
Other:
- note added: "5V 5A"
